File: Circuit/WallGrinder.brd (EAGLE design)
At the start: 95.2 x 94.9 mm, 32 parts, among them IC2 MIC5225-5v, J5 1X04_SMD_STRAIGHT_COMBO, J6 1X04_SMD_STRAIGHT_COMBO

Commit message: movement
Parts:
- moved LED4 3.88 mm to (30.4, 66.8)
Connections:
- new net N$3: LED01.2-DOUT, LED2.4-DIN
- net LED_IN: no longer LED01.2-DOUT, LED2.4-DIN
Routing:
- net GND: track 123.4 -> 0.00 mm, vias 9 -> 1
- net LED_IN: track 75.1 -> 29.4 mm
- net N$3: track 0.00 -> 35.9 mm, vias 0 -> 2
- net MOUT1_2: track 49.7 -> 78.2 mm, vias 0 -> 2
- net VCC: track 297.2 -> 273.0 mm, vias 5 -> 2
- net EOUT3_A: track 76.6 -> 53.0 mm, vias 2 -> 4
- net 5V: track 147.4 -> 126.1 mm
- net EOUT4_A: track 38.9 -> 57.4 mm, vias 2 -> 0
- net MPHASE_4: track 100.8 -> 82.9 mm, vias 0 -> 2
- net MENABLE_1: track 71.7 -> 89.1 mm
- net MPHASE_2: track 73.0 -> 87.5 mm, vias 2 -> 0
- net MOUT1_1: track 50.1 -> 41.7 mm
- net MPHASE_1: track 66.8 -> 74.9 mm
- net EOUT1_A: track 50.7 -> 58.5 mm, vias 4 -> 2
- net MPHASE_3: track 103.5 -> 110.2 mm
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